File: hackpad1.kicad_sch (KiCad schematic)
At the start: 0 parts

Commit message: Add buttons and microcontroller to schematic
Added all the buttons, diodes and microcontroller
Parts:
- added D1, D2, D3, D4, D5, D6, D7, D8: D, symbol Device:D
- added SW1, SW2, SW3, SW4, SW5, SW6, SW7, SW8: SW_Push, symbol Switch:SW_Push
- added U1: MOUDLE-SEEEDUINO-XIAO, symbol XIAO_RP2040:MOUDLE-SEEEDUINO-XIAO
Connections:
- new net: D5.2 (A), SW5.1
- new net: SW1.2, SW5.2
- new net: D5.1 (K), D6.1 (K), D7.1 (K), D8.1 (K)
- new net: D6.2 (A), SW6.1
- new net: D4.2 (A), SW4.1
- new net: SW4.2, SW8.2
- new net: D1.2 (A), SW1.1
- new net: D1.1 (K), D2.1 (K), D3.1 (K), D4.1 (K)
- new net: D3.2 (A), SW3.1
- new net: D8.2 (A), SW8.1
- new net: D7.2 (A), SW7.1
- new net: SW3.2, SW7.2
- new net: D2.2 (A), SW2.1
- new net: SW2.2, SW6.2
- new net +5V: U1.14 (5V)
- new net GND: U1.13 (GND)

Commit message: Finish schematic
Finished schematic
Parts:
- added D10, D9: SK6812MINI-E, SK6812MINI-E - 3.2x2.8x1.78mm, symbol Neopixel_hackpad:SK6812MINI-E
Connections:
- net +5V: now also D10.1 (VDD), D9.1 (VDD)
- net GND: now also D10.3 (VSS), D9.3 (VSS)
- net COL1: now reaches SW1.2, SW5.2
- net COL1: now also U1.4 (PA11_A3_D3), U1.5 (PA8_A4_D4_SDA), U1.6 (PA9_A5_D5_SCL), U1.7 (PB08_A6_D6_TX)
- net ROW2: now reaches D5.1 (K), D6.1 (K), D7.1 (K), D8.1 (K)
- net ROW2: now also U1.3 (PA10_A2_D2)
- net ROW1: now reaches U1.2 (PA4_A1_D1)
- net ROW1: now also D1.1 (K), D2.1 (K), D3.1 (K), D4.1 (K)
- net COL4: now reaches SW4.2, SW8.2
- net COL3: now reaches SW3.2, SW7.2
- net COL2: now reaches SW2.2, SW6.2
- new net: D10.4 (DIN), D9.2 (DOUT)
- new net NEO: D9.4 (DIN)
Other:
- moved on the sheet: D1, D2, D3, D4, D5, D6, D7, D8, SW1, SW2, SW3, SW4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
